File: _autosave-horizon.kicad_pcb (KiCad board)
At the start: 4 copper layers, 50 x 100 mm, 263 parts, among them IC1 A3909, J1 Micro_SD_Card_Det1, J10 Conn_01x02_Pin, J11 USB_C_Receptacle_USB2.0_16P, J12 Conn_01x04, J13 1x3 servo, J14 1x3 servo, J15 arming terminal, J16 arming terminal, J17 arming terminal, J18 arming terminal, J19 Screw_Terminal_01x02, J2 Conn_02x03_Counter_Clockwise, J20 Screw_Terminal_01x02, J21 Screw_Terminal_01x02, J22 Screw_Terminal_01x02, J23 USB_C_Receptacle_USB2.0_16P, J24 USB_C_Receptacle_USB2.0_16P, J25 Conn_Coaxial, J3 Conn_Coaxial, J5 Screw_Term, J6 1x3 servo, J7 Conn_02x03_Counter_Clockwise, J8 Conn_02x03_Counter_Clockwise, J9 1x3 servo, Q1 IRLML6402, Q10 IRLML6402, Q11 IRLML6402, Q2 DMG2301L, Q3 IRLML6402, Q4 IRLML6402, Q5 IRLML6402, Q6 IRLML6402, Q7 BSS138, Q8 IRLML6402, Q9 IRLML6402, U1 MMCU, U10 LSM6DS3, U11 BGM220SC12WGA2R, U12 PE4259, U13 LTC4412xS6, U14 TPS61092, U15 AP2112K-3.3, U2 IMU, U3 NMCU, U4 TMCU, U5 LPS22HB, U6 GPS, U7 SX1276, U8 NAND, U9 TPS82130, Y1 Crystal, Y2 32.768kHz, Y4 32MHz

Commit message: wiring
Parts:
- moved R72 2.92 mm to (59.9, 108.8), turned to 0 degrees
- moved TP16 1.96 mm to (85.2, 99.8)
- moved REF** 1.22 mm to (57.9, 112.8)
- moved C18 0.75 mm to (76.1, 91.7)
- moved Q7 0.56 mm to (59.4, 106.0)
- moved R46 0.45 mm to (89.5, 93.3)
- moved U15 0.41 mm to (87.0, 90.2)
- moved C34 0.38 mm to (91.1, 92.6)
- moved D21 0.20 mm to (90.0, 95.8)
- moved D22 0.12 mm to (90.8, 98.6)
- moved R47 0.11 mm to (89.2, 98.3)
- moved L2 0.09 mm to (95.5, 99.7)
- turned C20 to 0 degrees
Connections:
- R79 pad 1: mosfet1_signal -> mosfet1_signalfire
- R81 pad 1: mosfet2_signal -> mosfet2_signalfire
- R83 pad 1: mosfet3_signal -> mosfet3_signalfire
- R85 pad 1: mosfet4_signal -> mosfet4_signalfire
- U3 pad 20: unconnected-(U3-PA11-Pad20) -> mosfet1_signalfire
- U3 pad 29: unconnected-(U3-PA12-Pad29) -> mosfet2_signalfire
- U3 pad 30: unconnected-(U3-PA13-Pad30) -> mosfet3_signalfire
- U3 pad 35: unconnected-(U3-PA16-Pad35) -> mosfet4_signalfire
Routing:
- net GND: track 8.20 -> 158.5 mm, vias 0 -> 93
- net 3B: track 0.00 -> 89.9 mm, vias 0 -> 1
- net 3R: track 0.00 -> 88.8 mm, vias 0 -> 1
- net 3G: track 0.00 -> 87.8 mm, vias 0 -> 1
- net Net-(D2-A): track 0.00 -> 81.5 mm, vias 0 -> 5
- net VBUS: track 0.00 -> 79.6 mm, vias 0 -> 4
- net D- DMCU-2: track 12.1 -> 70.9 mm, vias 1 -> 2
- net D+ DMCU-2: track 15.7 -> 71.3 mm, vias 1 -> 2
- net D- MMCU: track 10.2 -> 62.3 mm, vias 1 -> 2
- net D+ DMCU-1: track 13.6 -> 65.1 mm, vias 1 -> 2
- net D- DMCU-1: track 12.4 -> 63.5 mm, vias 1 -> 2
- net D+ MMCU: track 14.5 -> 63.9 mm, vias 1 -> 2
- net +3.3V: track 26.6 -> 50.6 mm, vias 0 -> 7
- net Net-(D6-K): track 0.00 -> 8.71 mm
- net Net-(D5-K): track 0.00 -> 8.67 mm
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