File: horizon-backups/horizon-2025-05-15_191045/horizon_1.kicad_sch (KiCad schematic)
At the start: 36 parts, among them J2 Conn_02x03_Counter_Clockwise, J7 Conn_02x03_Counter_Clockwise, J8 Conn_02x03_Counter_Clockwise, U1 MMCU, U3 NMCU, U4 TMCU, Y1 Crystal

Commit message: ERC Changes
Parts:
- removed C59, C60, C61, C62: 100nF, symbol Device:C
Connections:
- net +3.3V: no longer C1.2, C10.2, C11.2, C12.2, C13.2, C17.2, C2.2, C3.1, C4.1, C5.1, C6.1, C7.2, C8.2, C9.2, J2.3 (Pin_3), J7.3 (Pin_3), J8.3 (Pin_3), U1.10 (A10/ADC0_DM0), U1.14 (VREF-H), U1.15 (VREF-L), U1.16 (VSSA), U1.17 (VREF_OUT), U1.31 (VSS), U1.4 (VSS), U1.47 (VSS), U3.22 (GND), U3.33 (GND), U3.47 (GND), U3.54 (GND), U3.7 (GNDANA), U4.22 (GND), U4.33 (GND), U4.47 (GND), U4.54 (GND), U4.7 (GNDANA)
- net PTA12: no longer U4.50 (PB23)
- net PTD4: no longer U3.49 (PB22)
- net GND: now reaches U3.55 (VDDCORE)
- net GND: now also C1.2, C10.2, C11.2, C12.2, C13.2, C17.2, C2.2, C3.1, C4.1, C5.1, C6.1, C7.2, C8.2, C9.2, J2.3 (Pin_3), J7.3 (Pin_3), J8.3 (Pin_3), U1.10 (A10/ADC0_DM0), U1.14 (VREF-H), U1.15 (VREF-L), U1.16 (VSSA), U1.17 (VREF_OUT), U1.31 (VSS), U1.4 (VSS), U1.47 (VSS), U3.22 (GND), U3.33 (GND), U3.47 (GND), U3.54 (GND), U3.7 (GNDANA), U4.22 (GND), U4.33 (GND), U4.47 (GND), U4.54 (GND), U4.55 (VDDCORE)
- net CS TMCU renamed Baro_int TMCU
- net RS_GPS TMCU: no longer names the net of U3.64 (PB03)
- net SPI0_SCK MMCU renamed  SPI0_SCK MMCU
- no-connect marks 98 -> 3
