File: horizon-backups/horizon-2025-05-15_191045/power.kicad_sch (KiCad schematic)
At the start: 47 parts, among them J10 Conn_01x02_Pin, Q2 DMG2301L, U12 TPS63061, U13 LTC4412xS6, U14 TPS61092, U15 AP2112K-3.3, U16 TPS61092, U9 TPS82130

Commit message: ERC Changes
Connections:
- net at C34.1, C35.1, R44.1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: no longer U15.3 (EN)
- net at U13.4 (STAT): now also U9.1 (EN)
- net at C32.1, D20.1 (K), U9.2 (VIN): no longer U9.1 (EN)
- net at U9.7 (PG): now also U15.3 (EN)
- no-connect marks 6 -> 0
