File: horizon-backups/horizon-2025-05-15_191045/sensor.kicad_sch (KiCad schematic)
At the start: 122 parts, among them IC1 A3909, J1 Micro_SD_Card_Det1, J13 1x3 servo, J14 1x3 servo, J15 arming terminal, J16 arming terminal, J17 arming terminal, J18 arming terminal, J19 Screw_Terminal_01x02, J20 Screw_Terminal_01x02, J21 Screw_Terminal_01x02, J22 Screw_Terminal_01x02, J3 Conn_Coaxial, J4 H9161TR-ND, J5 Screw_Term, J6 1x3 servo, J9 1x3 servo, Q1 2N7002, Q10 2N7002, Q11 2N7002, Q12 2N7002, Q13 2N7002, Q3 2N7002, Q4 2N7002, Q5 2N7002, Q6 2N7002, Q7 BSS138, U10 LSM6DS3, U2 IMU, U5 LPS22HB, U6 GPS, U7 SX1276, U8 NAND, Y2 32.768kHz

Commit message: ERC Changes
Connections:
- net RS_GPS TMCU renamed ANY GPIO PIN
- no-connect marks 32 -> 13
Changed lines of the file:
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@@
-	)
-	(no_connect
-		(at 76.2 154.94)
 	)
 	(no_connect
@@
 	)
 	(no_connect
-		(at 262.89 38.1)
-	)
-	(no_connect
-		(at 106.68 157.48)
-	)
-	(no_connect
-		(at 76.2 144.78)
-	)
-	(no_connect
-		(at 76.2 160.02)
-	)
-	(no_connect
-		(at 76.2 167.64)
-	)
-	(no_connect
 		(at 227.33 151.13)
 	)
@@
 	)
 	(no_connect
-		(at 106.68 170.18)
-	)
-	(no_connect
-		(at 325.12 52.07)
-	)
-	(no_connect
 		(at 93.98 54.61)
-	)
-	(no_connect
-		(at 201.93 58.42)
-	)
-	(no_connect
-		(at 325.12 49.53)
 	)
 	(no_connect
@@
 	)
 	(no_connect
-		(at 33.02 167.64)
-	)
-	(no_connect
 		(at 106.68 154.94)
 	)
@@
 	)
 	(no_connect
-		(at 33.02 170.18)
-	)
-	(no_connect
 		(at 48.26 57.15)
-	)
-	(no_connect
-		(at 76.2 142.24)
 	)
 	(no_connect
@@
 	)
 	(no_connect
-		(at 76.2 162.56)
-	)
-	(no_connect
-		(at 76.2 139.7)
-	)
-	(no_connect
-		(at 76.2 157.48)
-	)
-	(no_connect
 		(at 48.26 54.61)
-	)
-	(no_connect
-		(at 262.89 40.64)
-	)
-	(no_connect
-		(at 106.68 162.56)
-	)
-	(no_connect
-		(at 355.6 41.91)
 	)
 	(bus_entry
@@
 		)
 	)
-	(global_label "RS_GPS TMCU"
+	(global_label "ANY GPIO PIN"
 		(shape input)
 		(at 40.64 41.91 180)
@@
 		)
 		(property "Intersheetrefs" "${INTERSHEET_REFS}"
-			(at 24.4711 41.91 0)
-			(effects
-				(font
+			(at 24.5313 41.91 0)
+			(effects
+				(font
