File: horizon-backups/horizon-2025-05-15_191045/usb.kicad_sch (KiCad schematic)
At the start: 21 parts, among them J11 USB_C_Receptacle_USB2.0_16P, SW1 SW_Rotary_1x4_MP, SW2 SW_Rotary_1x4_MP

Commit message: ERC Changes
Connections:
- no-connect marks 6 -> 2
Changed lines of the file:
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@@
-	)
-	(no_connect
-		(at 167.64 63.5)
 	)
 	(no_connect
@@
 	)
 	(no_connect
-		(at 177.8 52.07)
-	)
-	(no_connect
 		(at 81.28 80.01)
 	)
-	(no_connect
-		(at 182.88 63.5)
-	)
-	(no_connect
-		(at 162.56 52.07)
-	)
 	(wire
