File: pcbway version *LOOKS ONLY*/horizon.kicad_pcb (KiCad board)
At the start: 4 copper layers, 50 x 100 mm, 209 parts, among them IC1 A3909, J1 Micro_SD_Card_Det1, J10 Conn_01x02_Pin, J11 USB_C_Receptacle_USB2.0_16P, J12 Conn_01x04, J13 1x3 servo, J14 1x3 servo, J15 arming terminal, J16 arming terminal, J19 Screw_Terminal_01x02, J20 Screw_Terminal_01x02, J4 H9161TR-ND, J5 Screw_Term, J6 1x3 servo, J9 1x3 servo, Q1 IRLML6402, Q2 DMG2301L, Q3 IRLML6402, Q4 IRLML6402, Q5 IRLML6402, Q6 IRLML6402, Q7 BSS138, Q8 IRLML6402, Q9 IRLML6402, SW1 SW_SP3T, SW2 SW_SP3T, U1 MMCU, U10 LSM6DS3, U11 BGM220SC12WGA2R, U12 PE4259, U13 LTC4412xS6, U14 TPS61092, U15 AP2112K-3.3, U3 NMCU, U4 TMCU, U5 LPS22HB, U6 GPS, U7 SX1276, U8 NAND, U9 TPS82130, Y1 Crystal, Y4 32MHz

Commit message: logo placement stuff
Parts:
- moved G*** 55.4 mm to (89.8, 28.5)
- moved G*** 3.13 mm to (82.1, 90.9)
Routing:
- net +3.3V: track 593.6 -> 611.9 mm, vias 57 -> 58
- net SWDIO DMCU-1: track 10.3 -> 17.8 mm
- net nRESET MMCU: track 24.5 -> 31.9 mm
- net SWCLK MMCU: track 35.7 -> 42.1 mm
- net nRESET DMCU-1: track 21.8 -> 27.9 mm
- net SWCLK DMCU-1: track 37.3 -> 43.1 mm
- net SWDIO MMCU: track 28.6 -> 34.3 mm
- net nRESET DMCU-2: track 19.6 -> 23.7 mm
- net SWCLK DMCU-2: track 17.7 -> 20.5 mm
- net SWDIO DMCU-2: track 18.5 -> 20.7 mm, vias 3 -> 4
Other:
- outline, holes or cut-outs redrawn
