File: flight computer/sensor.kicad_sch (KiCad schematic)
At the start: 131 parts, among them IC1 A3909, J1 Micro_SD_Card_Det1, J12 Conn_01x04, J13 1x3 servo, J14 1x3 servo, J15 arming terminal, J16 arming terminal, J17 H9161TR-ND, J19 Screw_Terminal_01x02, J20 Screw_Terminal_01x02, J3 H9161TR-ND, J4 H9161TR-ND, J5 Screw_Term, J6 1x3 servo, J9 1x3 servo, Q1 IRLML6402, Q3 IRLML6402, Q4 IRLML6402, Q5 IRLML6402, Q6 IRLML6402, Q7 BSS138, Q8 IRLML6402, Q9 IRLML6402, U10 LSM6DS3, U11 BGM220SC12WGA2R, U12 PE4259, U5 LPS22HB, U6 GPS, U7 SX1276, U8 NAND, Y4 32MHz

Commit message: Wired the headers for programming 3 MCU'S + some footprint fixes and additions for photos:(
Parts:
- J17, J3, J4: footprint U.FL-R-SMT_01_:HRS_U.FL-R-SMT_01_ -> U.FL:HRS_U.FL-R-SMT_01_
- U11: footprint KiCADv6:BGM220SC12WGA2R -> BGM220SC12WGA2R:BGM220SC12WGA2R
Changed lines of the file:
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@@
 			)
 		)
-		(property "Footprint" "U.FL-R-SMT_01_:HRS_U.FL-R-SMT_01_"
+		(property "Footprint" "U.FL:HRS_U.FL-R-SMT_01_"
 			(at 114.3 49.53 0)
 			(effects
@@
 			)
 		)
-		(property "Footprint" "KiCADv6:BGM220SC12WGA2R"
+		(property "Footprint" "BGM220SC12WGA2R:BGM220SC12WGA2R"
 			(at -83.82 81.28 0)
 			(effects
@@
 			)
 		)
-		(property "Footprint" "U.FL-R-SMT_01_:HRS_U.FL-R-SMT_01_"
+		(property "Footprint" "U.FL:HRS_U.FL-R-SMT_01_"
 			(at -49.53 196.85 0)
 			(effects
@@
 			)
 		)
-		(property "Footprint" "U.FL-R-SMT_01_:HRS_U.FL-R-SMT_01_"
+		(property "Footprint" "U.FL:HRS_U.FL-R-SMT_01_"
 			(at -8.89 91.44 0)
 			(effects
