File: flight computer/sensor.kicad_sch (KiCad schematic)
At the start: 92 parts, among them J1 Micro_SD_Card_Det1, J12 Conn_01x04, J13 1x3 servo, J14 1x3 servo, J15 arming terminal, J16 arming terminal, J17 H9161TR-ND, J19 Screw_Terminal_01x02, J20 Screw_Terminal_01x02, J3 H9161TR-ND, J4 H9161TR-ND, J5 Screw_Term, J6 1x3 servo, J9 1x3 servo, Q7 BSS138, Q8 IRLML6402, Q9 IRLML6402, U10 LSM6DS3, U11 BGM220SC12WGA2R, U16 SX1262IMLTRT, U17 PE4259, U5 LPS22HB, U6 GPS, U8 NAND, Y2 32MHz

Commit message: added BGM220SC12WGA2R
Parts:
- J17, J3, J4: footprint U.FL-R-SMT_01_:HRS_U.FL-R-SMT_01_ -> Connector_Coaxial:U.FL_Hirose_U.FL-R-SMT-1_Vertical
- U11: footprint BGM220SC12WGA2R:BGM220SC12WGA2R -> BGM220SC12WGA2R:BGM220S_SIL
Changed lines of the file:
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@@
 			)
 		)
-		(property "Footprint" "U.FL-R-SMT_01_:HRS_U.FL-R-SMT_01_"
+		(property "Footprint" "Connector_Coaxial:U.FL_Hirose_U.FL-R-SMT-1_Vertical"
 			(at 114.3 49.53 0)
 			(effects
@@
 			)
 		)
-		(property "Footprint" "BGM220SC12WGA2R:BGM220SC12WGA2R"
+		(property "Footprint" "BGM220SC12WGA2R:BGM220S_SIL"
 			(at -83.82 81.28 0)
 			(effects
@@
 			)
 		)
-		(property "Footprint" "U.FL-R-SMT_01_:HRS_U.FL-R-SMT_01_"
+		(property "Footprint" "Connector_Coaxial:U.FL_Hirose_U.FL-R-SMT-1_Vertical"
 			(at -7.62 232.41 0)
 			(effects
@@
 			)
 		)
-		(property "Footprint" "U.FL-R-SMT_01_:HRS_U.FL-R-SMT_01_"
+		(property "Footprint" "Connector_Coaxial:U.FL_Hirose_U.FL-R-SMT-1_Vertical"
 			(at -8.89 91.44 0)
 			(effects

Commit message: force push :'/
Connections:
- net SD_DETECT: no longer J1.9 (DET), R56.2
- new net: J1.9 (DET), R56.2
Other:
- moved on the sheet: C15, J1, R12, R54, R55, R56, U8

Commit message: added buzzer footprint
Parts:
- BZ2: footprint (none) -> Buzzer:MLT-8530_JHE
Changed lines of the file:
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@@
 			)
 		)
-		(property "Footprint" ""
+		(property "Footprint" "Buzzer:MLT-8530_JHE"
 			(at 35.56 88.9 0)
 			(effects

Commit message: DONE DONE FUCKING DONE
Connections:
- net Earth is gone; now on net GND: C14.1, C37.1, C38.2, C39.1, C40.2, C46.2, C47.2, C48.2, FL1.10 (GND), FL1.2 (GND), FL1.5 (GND), FL1.7 (GND), FL1.9 (GND), U16.2 (GND), U16.20 (GND), U16.25 (GND), U16.5 (GND), U16.8 (GND), U17.2 (GND), Y2.2, Y2.4

Commit message: push
Parts:
- added C23, C26: C, symbol Device:C
- added R15, R16: R, symbol Device:R
Connections:
- net GND: now also C26.2, R15.1, R16.1
- net at J5.1 (Pin_1): now also C23.1
- net at J5.2 (Pin_2): now also C23.2
Other:
- moved on the sheet: J5

Commit message: everything everything :) wait no i still havent added the secondary rotary encoder dont push
Parts:
- removed C23, C26: C, symbol Device:C
- removed R15, R16: R, symbol Device:R
Connections:
- net +5V: now also J5.1 (Pin_1)
- net GND: now also J5.2 (Pin_2)
- net at D4.1 (K), Q9.2 (S): now also J20.2 (Pin_2)
- net at J20.1 (Pin_1): now also F2.1
Other:
- moved on the sheet: J5

Commit message: if this breaks stuff womp womp
Parts:
- removed R1, R2: 10 kΩ, Resistor_SMD:R_0603_1608Metric, symbol Device:R
Connections:
- net +3.3V: no longer U11.33 (PC05), U11.35 (RESETn)
- net BGM_INT: now also U11.33 (PC05)
- net BGM_RESET: now also U11.35 (RESETn)
Other:
- note added: "-note: removed attempted pullups-"
- note added: "NOTE/TODO : ADD SWD HEADER FOR BLUETOOTH NEED SWD FOR CONFIG"
