File: flight computer/_autosave-horizon.kicad_pcb (KiCad board)
At the start: 4 copper layers, 50.8 x 95.7 mm, 193 parts, among them IC1 A3909, J1 Micro_SD_Card_Det1, J10 Conn_01x02_Pin, J11 USB_C_Receptacle_USB2.0_16P, J12 Conn_01x04, J13 1x3 servo, J14 1x3 servo, J15 arming terminal, J16 arming terminal, J17 H9161TR-ND, J18 Conn_02x03_Counter_Clockwise, J19 Screw_Terminal_01x02, J2 Conn_02x03_Counter_Clockwise, J20 Screw_Terminal_01x02, J21 Conn_02x03_Counter_Clockwise, J3 H9161TR-ND, J4 H9161TR-ND, J5 Screw_Term, J6 1x3 servo, J7 Conn_02x03_Counter_Clockwise, J8 Conn_02x03_Counter_Clockwise, J9 1x3 servo, Q1 IRLML6402, Q2 DMG2301L, Q3 IRLML6402, Q4 IRLML6402, Q5 IRLML6402, Q6 IRLML6402, Q7 BSS138, Q8 IRLML6402, Q9 IRLML6402, SW1 CK_KMS2xxG, U1 MMCU, U10 LSM6DS3, U13 LTC4412xS6, U14 TPS61092, U15 AP2112K-3.3, U16 SX1262IMLTRT, U17 PE4259, U2 MKL02Z32VFG4, U5 LPS22HB, U6 GPS, U8 NAND, U9 TPS82130, Y1 Crystal, Y2 32MHz

Commit message: random push
Parts:
- moved F2 15.3 mm to (224.3, 38.1)
- moved F1 12.6 mm to (174.4, 37.6), turned to 0 degrees
- moved R81 10.7 mm to (220.8, 39.6), turned to -90 degrees
- moved R59 3.87 mm to (209.3, 44.3)
- moved R80 3.86 mm to (212.3, 44.3)
- moved Q9 1.61 mm to (211.8, 41.6), turned to -90 degrees
- moved D4 0.80 mm to (209.3, 42.0)
Connections:
- F2 pad 1: Net-(J20-Pin_2) -> Net-(J20-Pin_1)
- J16 pad 1: +5V -> Net-(J16-Pin_1)
- J16 pad 2: Net-(J16-Pin_2) -> +5V
- J20 pad 1: Net-(D4-K) -> Net-(J20-Pin_1)
- J20 pad 2: Net-(J20-Pin_2) -> Net-(D4-K)
- R80 pad 1: Net-(J16-Pin_2) -> Net-(J16-Pin_1)
Routing:
- net Net-(Q9-D): track 2.55 -> 8.04 mm
- net Net-(J16-Pin_2): track 4.06 -> 0.00 mm
- net (no net): track 0.00 -> 4.06 mm
- net Net-(D4-K): track 0.00 -> 3.43 mm
- net Net-(J19-Pin_2): track 0.00 -> 2.19 mm
- net Net-(J20-Pin_1): track 0.00 -> 2.04 mm
