File: flight computer/_autosave-horizon.kicad_pcb (KiCad board)
At the start: 4 copper layers, 50.8 x 95.7 mm, 85 parts, among them J1 Micro_SD_Card_Det1, J10 Conn_01x02_Pin, J11 USB_C_Receptacle_USB2.0_16P, J12 Conn_01x04, J13 1x3 servo, J14 1x3 servo, J15 arming terminal, J16 arming terminal, J18 Conn_02x03_Counter_Clockwise, J19 Screw_Terminal_01x02, J20 Screw_Terminal_01x02, J21 Conn_02x03_Counter_Clockwise, J3 H9161TR-ND, J5 Screw_Term, J6 1x3 servo, J8 Conn_02x03_Counter_Clockwise, J9 1x3 servo, Q2 DMG2301L, SW1 CK_KMS2xxG, U1 MMCU, U10 LSM6DS3, U13 LTC4412xS6, U14 TPS61092, U15 AP2112K-3.3, U16 SX1262IMLTRT, U2 MKL02Z32VFG4, U5 LPS22HB, U6 GPS, U8 NAND, U9 TPS82130, Y1 Crystal

Commit message: power + usbc
Parts:
- moved D8 72.2 mm to (199.4, 35.0)
- moved R47 36.9 mm to (223.1, 41.3)
- moved D22 36.9 mm to (220.8, 40.3)
- moved D21 30.2 mm to (203.9, 37.1), turned to 0 degrees
- moved C35 28.4 mm to (206.9, 38.3), turned to 180 degrees
- moved R46 27.0 mm to (206.9, 36.8), turned to 180 degrees
- moved C33 26.8 mm to (203.8, 32.2), turned to 0 degrees
- moved C36 26.5 mm to (200.5, 39.9)
- moved U15 26.5 mm to (203.3, 39.7)
- moved U9 25.7 mm to (203.6, 34.7)
- moved R44 25.2 mm to (206.1, 34.5)
- moved R45 25.2 mm to (206.9, 32.2)
- moved C34 25.2 mm to (207.7, 34.5)
- moved D20 24.7 mm to (197.9, 34.2)
- moved C32 24.7 mm to (201.0, 33.4)
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Routing:
- net Net-(U15-EN): track 0.00 -> 14.2 mm
- net bat: track 7.30 -> 17.5 mm
- net POWAAAA: track 7.02 -> 17.2 mm
- net Net-(L2-Pad2): track 0.00 -> 7.48 mm
- net Net-(U9-FB): track 0.00 -> 4.15 mm
- net GND: track 10.6 -> 14.4 mm, vias 0 -> 3
- net Net-(Q2-G): track 0.00 -> 1.98 mm
- net +5V: track 0.00 -> 1.70 mm
- net Net-(D21-A): track 0.00 -> 1.57 mm
- net Net-(U9-SS/TR): track 0.00 -> 1.57 mm
