File: flight computer/horizon.kicad_pcb (KiCad board)
At the start: 4 copper layers, 50.8 x 95.7 mm, 151 parts, among them J1 Micro_SD_Card_Det1, J10 Conn_01x02_Pin, J11 USB_C_Receptacle_USB2.0_16P, J12 Conn_01x04, J13 1x3 servo, J14 1x3 servo, J15 arming terminal, J16 arming terminal, J17 H9161TR-ND, J18 Conn_02x03_Counter_Clockwise, J19 Screw_Terminal_01x02, J20 Screw_Terminal_01x02, J21 Conn_02x03_Counter_Clockwise, J3 H9161TR-ND, J4 H9161TR-ND, J5 Screw_Term, J6 1x3 servo, J9 1x3 servo, Q2 DMG2301L, Q7 BSS138, Q8 IRLML6402, Q9 IRLML6402, SW1 CK_KMS2xxG, U1 MMCU, U10 LSM6DS3, U11 BGM220SC12WGA2R, U13 LTC4412xS6, U15 AP2112K-3.3, U16 SX1262IMLTRT, U17 PE4259, U2 MKL02Z32VFG4, U3 TPS61200DRC, U5 LPS22HB, U6 GPS, U8 NAND, U9 TPS82130, Y1 Crystal, Y2 32MHz

Commit message: now you can continue
Parts:
- moved U5 37.5 mm to (208.2, 62.2)
- moved C50 37.5 mm to (208.0, 60.2)
- moved R39 37.5 mm to (210.3, 63.7)
- moved R52 37.5 mm to (211.0, 61.4), turned to 180 degrees
- moved R53 37.5 mm to (208.8, 65.0)
- moved C51 37.5 mm to (206.2, 62.6)
Routing:
- net CS_BARO TMCU: track 0.00 -> 1.44 mm
- net Net-(U5-INT_DRDY): track 0.00 -> 1.44 mm
Changed lines of the file:
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@@
 	(footprint "Capacitor_SMD:C_0603_1608Metric"
 		(layer "F.Cu")
-		(at 190.77 96.755 90)
+		(at 206.19 62.585 90)
 		(descr "Capacitor SMD 0603 (1608 Metric), square (rectangular) end terminal, IPC-7351 nominal, (Body size source: IPC-SM-782 page 76, https://www.pcb-3d.com/wordpress/wp-content/uploads/ipc-sm-782a_amendment_1_and_2.pdf), generated with kicad-footprint-generator")
 		(tags "capacitor")
@@
 	(footprint "Capacitor_SMD:C_0603_1608Metric"
 		(layer "F.Cu")
-		(at 192.555 94.37 180)
+		(at 207.975 60.2 180)
 		(descr "Capacitor SMD 0603 (1608 Metric), square (rectangular) end terminal, IPC-7351 nominal, (Body size source: IPC-SM-782 page 76, https://www.pcb-3d.com/wordpress/wp-content/uploads/ipc-sm-782a_amendment_1_and_2.pdf), generated with kicad-footprint-generator")
 		(tags "capacitor")
@@
 			(at 0 -1.43 0)
 			(layer "F.SilkS")
+			(hide yes)
 			(effects
 				(font
@@
 	(footprint "Resistor_SMD:R_0603_1608Metric"
 		(layer "F.Cu")
-		(at 193.34 99.205 90)
+		(at 208.76 65.035 90)
 		(descr "Resistor SMD 0603 (1608 Metric), square (rectangular) end terminal, IPC-7351 nominal, (Body size source: IPC-SM-782 page 72, https://www.pcb-3d.com/wordpress/wp-content/uploads/ipc-sm-782a_amendment_1_and_2.pdf), generated with kicad-footprint-generator")
 		(tags "resistor")
@@
 	(footprint "Package_LGA:ST_HLGA-10_2x2mm_P0.5mm_LayoutBorder3x2y"
 		(layer "F.Cu")
-		(at 192.8175 96.42)
+		(at 208.2375 62.25)
 		(descr "ST  HLGA, 10 Pin (https://www.st.com/resource/en/datasheet/lps22hh.pdf#page=55), generated with kicad-footprint-generator ipc_noLead_generator.py")
 		(tags "ST HLGA NoLead")
@@
 			(at 0 -1.95 0)
 			(layer "F.SilkS")
+			(hide yes)
 			(effects
 				(font
@@
 	(footprint "Resistor_SMD:R_0603_1608Metric"
 		(layer "F.Cu")
-		(at 194.86 97.885 90)
+		(at 210.28 63.715 90)
 		(descr "Resistor SMD 0603 (1608 Metric), square (rectangular) end terminal, IPC-7351 nominal, (Body size source: IPC-SM-782 page 72, https://www.pcb-3d.com/wordpress/wp-content/uploads/ipc-sm-782a_amendment_1_and_2.pdf), generated with kicad-footprint-generator")
 		(tags "resistor")
@@
 			(at 0 -1.43 90)
 			(layer "F.SilkS")
+			(hide yes)
 			(effects
 				(font
@@
 	(footprint "Resistor_SMD:R_0603_1608Metric"
 		(layer "F.Cu")
-		(at 195.61 95.61)
+		(at 211.03 61.44 180)
 		(descr "Resistor SMD 0603 (1608 Metric), square (rectangular) end terminal, IPC-7351 nominal, (Body size source: IPC-SM-782 page 72, https://www.pcb-3d.com/wordpress/wp-content/uploads/ipc-sm-782a_amendment_1_and_2.pdf), generated with kicad-footprint-generator")
 		(tags "resistor")
@@
 		(attr smd)
 		(fp_line
-			(start -0.237258 -0.5225)
-			(end 0.237258 -0.5225)
+			(start -0.237258 0.5225)
+			(end 0.237258 0.5225)
 			(stroke
 				(width 0.12)
@@
 		)
 		(fp_line
-			(start -0.237258 0.5225)
-			(end 0.237258 0.5225)
+			(start -0.237258 -0.5225)
+			(end 0.237258 -0.5225)
 			(stroke
 				(width 0.12)
@@
 		)
 		(fp_line
-			(start -1.48 -0.73)
-			(end 1.48 -0.73)
+			(start 1.48 0.73)
+			(end -1.48 0.73)
 			(stroke
 				(width 0.05)
@@
 		)
 		(fp_line
-			(start -1.48 0.73)
-			(end -1.48 -0.73)
+			(start 1.48 -0.73)
+			(end 1.48 0.73)
 			(stroke
 				(width 0.05)
@@
 		)
 		(fp_line
-			(start 1.48 -0.73)
-			(end 1.48 0.73)
+			(start -1.48 0.73)
+			(end -1.48 -0.73)
 			(stroke
 				(width 0.05)
@@
 		)
 		(fp_line
-			(start 1.48 0.73)
-			(end -1.48 0.73)
+			(start -1.48 -0.73)
+			(end 1.48 -0.73)
 			(stroke
 				(width 0.05)
@@
 		)
 		(fp_line
-			(start -0.8 -0.4125)
-			(end 0.8 -0.4125)
+			(start 0.8 0.4125)
+			(end -0.8 0.4125)
 			(stroke
 				(width 0.1)
@@
 		)
 		(fp_line
-			(start -0.8 0.4125)
-			(end -0.8 -0.4125)
+			(start 0.8 -0.4125)
+			(end 0.8 0.4125)
 			(stroke
 				(width 0.1)
@@
 		)
 		(fp_line
-			(start 0.8 -0.4125)
-			(end 0.8 0.4125)
+			(start -0.8 0.4125)
+			(end -0.8 -0.4125)
 			(stroke
 				(width 0.1)
@@
 		)
 		(fp_line
-			(start 0.8 0.4125)
-			(end -0.8 0.4125)
+			(start -0.8 -0.4125)
+			(end 0.8 -0.4125)
 			(stroke
 				(width 0.1)
@@
 		)
 		(pad "1" smd roundrect
-			(at -0.825 0)
+			(at -0.825 0 180)
 			(size 0.8 0.95)
 			(layers "F.Cu" "F.Mask" "F.Paste")
@@
 		)
 		(pad "2" smd roundrect
-			(at 0.825 0)
+			(at 0.825 0 180)
 			(size 0.8 0.95)
 			(layers "F.Cu" "F.Mask" "F.Paste")
@@
 	)
 	(segment
-		(start 193.3175 95.6575)
-		(end 193.3175 95.2225)
+		(start 208.7375 61.4875)
+		(end 208.7375 61.0525)
 		(width 0.2)
 		(layer "F.Cu")
@@
 	)
 	(segment
-		(start 191.52 97.53)
-		(end 191.7 97.35)
+		(start 206.94 63.36)
+		(end 207.12 63.18)
 		(width 0.2)
 		(layer "F.Cu")
@@
 	)
 	(segment
-		(start 192.8175 95.6575)
-		(end 193.3175 95.6575)
+		(start 208.2375 61.4875)
+		(end 208.7375 61.4875)
 		(width 0.2)
 		(layer "F.Cu")
@@
 	)
 	(segment
-		(start 190.77 97.53)
-		(end 191.52 97.53)
+		(start 206.19 63.36)
+		(end 206.94 63.36)
 		(width 0.2)
 		(layer "F.Cu")
@@
 	)
 	(segment
-		(start 192.3175 97.1825)
-		(end 191.8675 97.1825)
+		(start 207.7375 63.0125)
+		(end 207.2875 63.0125)
 		(width 0.2)
 		(layer "F.Cu")
@@
 	)
 	(segment
-		(start 193.33 94.37)
-		(end 193.33 95.21)
+		(start 208.75 60.2)
+		(end 208.75 61.04)
 		(width 0.2)
 		(layer "F.Cu")
@@
 	)
 	(segment
-		(start 191.8675 97.1825)
-		(end 191.7 97.35)
+		(start 207.2875 63.0125)
+		(end 207.12 63.18)
 		(width 0.2)
 		(layer "F.Cu")
@@
 	)
 	(segment
-		(start 193.3175 95.2225)
-		(end 193.33 95.21)
+		(start 208.7375 61.0525)
+		(end 208.75 61.04)
 		(width 0.2)
 		(layer "F.Cu")
@@
 	)
 	(via
-		(at 193.33 95.21)
+		(at 208.75 61.04)
 		(size 0.55)
 		(drill 0.3)
@@
 	)
 	(via
-		(at 191.7 97.35)
+		(at 207.12 63.18)
 		(size 0.55)
 		(drill 0.3)
@@
 	)
 	(segment
-		(start 192.3175 95.6575)
-		(end 192.3175 94.9075)
+		(start 207.7375 61.4875)
+		(end 207.7375 60.7375)
 		(width 0.2)
 		(layer "F.Cu")
@@
 	)
 	(segment
-		(start 192.3175 94.9075)
-		(end 191.78 94.37)
+		(start 207.7375 60.7375)
+		(end 207.2 60.2)
 		(width 0.2)
 		(layer "F.Cu")
@@
 	)
 	(segment
-		(start 190.96 96.17)
-		(end 190.77 95.98)
+		(start 206.38 62)
+		(end 206.19 61.81)
 		(width 0.2)
 		(layer "F.Cu")
@@
 	)
 	(segment
-		(start 192.3175 95.6575)
-		(end 192.3175 95.9075)
+		(start 207.7375 61.4875)
+		(end 207.7375 61.7375)
 		(width 0.2)
 		(layer "F.Cu")
@@
 	)
 	(segment
-		(start 192.055 96.17)
-		(end 190.96 96.17)
+		(start 207.475 62)
+		(end 206.38 62)
 		(width 0.2)
 		(layer "F.Cu")
@@
 	)
 	(segment
-		(start 192.3175 95.9075)
-		(end 192.055 96.17)
+		(start 207.7375 61.7375)
+		(end 207.475 62)
 		(width 0.2)
 		(layer "F.Cu")
@@
 	)
 	(segment
+		(start 209.39 62.89)
+		(end 209 62.5)
+		(width 0.2)
+		(layer "F.Cu")
+		(net 37)
+	)
+	(segment
+		(start 210.28 62.89)
+		(end 209.39 62.89)
+		(width 0.2)
+		(layer "F.Cu")
+		(net 37)
+	)
+	(segment
 		(start 170.260001 113.579999)
 		(end 170.73 113.11)
@@
 	)
 	(segment
-		(start 193.34 98.38)
-		(end 193.34 97.205)
+		(start 208.76 64.21)
+		(end 208.76 63.035)
 		(width 0.2)
 		(layer "F.Cu")
@@
 	)
 	(segment
-		(start 193.34 97.205)
-		(end 193.3175 97.1825)
+		(start 208.76 63.035)
+		(end 208.7375 63.0125)
 		(width 0.2)
 		(layer "F.Cu")
@@
 	)
 	(segment
+		(start 210.205 61.44)
+		(end 209.56 61.44)
+		(width 0.2)
+		(layer "F.Cu")
+		(net 219)
+	)
+	(segment
+		(start 209.56 61.44)
+		(end 209 62)
+		(width 0.2)
+		(layer "F.Cu")
+		(net 219)
+	)
+	(segment
