File: flight computer/_autosave-sensor.kicad_sch (KiCad schematic)
At the start: 91 parts, among them J1 Micro_SD_Card_Det1, J12 Conn_01x04, J13 1x3 servo, J14 1x3 servo, J15 arming terminal, J16 arming terminal, J17 H9161TR-ND, J19 Screw_Terminal_01x02, J20 Screw_Terminal_01x02, J22 Bluetooth Programming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

Commit message: bluetooth, gps, gyro reviewed - doing pressure tmrw
Other:
- note added: "Charlie's heart was pounding so hard he swore Luke could hear it over the hiss of the hydrogen tanks. The balloon above them strained against its tether, pale and glowing in the afternoon light, but all Charlie could see was Luke, crouched over the wiring, lips pressed together in concentration. "H-h-hi, L-luke," Charlie stammered, clipboard clutched to his chest like a shield. His cheeks were al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"
- note added: "I rushed to the canopy where the other teenagers were watching from afar and broke the news to them. The words hung in the air for a split second, before the low murmur of panic began to ripple through the group. Faces that were once full of excitement now wore masks of disbelief. I could hear snippets of frantic conversation: 'We can't be out of hydrogen!' 'This isn't happening.' 'What are we su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"
- moved on the sheet: R39
Changed lines of the file:
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@@
 		)
 	)
+	(text "Charlie's heart was pounding so hard he swore Luke could hear it over the hiss of the hydrogen tanks. The balloon above them strained against its tether, pale and glowing in the afternoon light, but all Charlie could see was Luke, crouched over the wiring, lips pressed together in concentration.\n\n\"H-h-hi, L-luke,\" Charlie stammered, clipboard clutched to his chest like a shield. His cheeks were already burning.\n\nLuke glanced up, the faintest smile tugging at the corner of his mouth. \"Hey, Charlie. You okay?\"\n\nCharlie nodded too quickly. \"Y-yeah, I-I'm fine. J-just… y-you know. Big day.\"\n\nLuke set down the circuit board and stood, brushing his palms against his jeans. He stepped closer-too close-and Charlie froze, every nerve lit up like a spark on live wire.\n\n\"You've been on edge all week,\" Luke said softly. \"It's not just the launch, is it?\"\n\nCharlie's throat went dry. He wanted to run, to bury his face in the grass, to disappear. Instead, words slipped out, cracked and trembling: \"I-it's you.\"\n\nLuke blinked. \"Me?\"\n\nCharlie's chest tightened. \"Y-yeah. Every time y-you talk, every time y-you look at me, I-I can't think straight.\" He laughed nervously, eyes darting away. \"N-not that I was ever really s-straight in the first place.\"\n\nFor a second, Charlie thought he'd ruined everything. Then Luke's hand brushed his, tentative but deliberate.\n\n\"I was hoping you'd say that,\" Luke whispered.\n\nCharlie's eyes snapped back to his. \"Y-you were?\"\n\nLuke nodded, leaning in until their foreheads almost touched. \"Charlie, I like you. I've liked you since the first time you tripped over your words in front of me.\"\n\nCharlie let out a shaky laugh, the weight of months lifting off his shoulders. \"Th-that happens a lot.\"\n\n\"Good,\" Luke murmured. \"Gives me more chances to fall for you.\"\n\nThe balloon tugged at its rope, eager to rise, but in that moment the world felt still. Charlie closed the space between them, his stutter dissolving into silence as their lips met-clumsy, desperate, but real.\n\nFor once, Charlie didn't care about the launch, the sponsors, or the science. All that mattered was Luke's hand in his, and the certainty that this was only the beginning."
+		(exclude_from_sim no)
+		(at 132.842 -100.076 0)
+		(effects
+			(font
+				(size 1.27 1.27)
+			)
+		)
+	)
 	(text "GPS"
 		(exclude_from_sim no)
@@
 		)
 	)
+	(text "I rushed to the canopy where the other teenagers were watching from afar and broke the news to them. The words hung in the air for a split second, before the low murmur of panic began to ripple through the group. Faces that were once full of excitement now wore masks of disbelief. I could hear snippets of frantic conversation: 'We can't be out of hydrogen!' 'This isn't happening.' 'What are we supposed to do?'\nThe balloon, still climbing higher with every minute, seemed almost oblivious to the chaos below. My stomach twisted. It felt like we were teetering on the edge of a cliff.\nCharlie was the first to turn to me, eyes wide. 'What now?' His voice was tight, like he was hoping I'd have some magical solution to this.\nI felt the weight of his gaze on me-the weight of everyone's hopes on me-and I knew I had to do something. Fast. But nothing came to mind. My head was spinning.\nI glanced back at the balloon, growing smaller by the second, and then I saw it-a flash of inspiration. The valve on the hydrogen tank. I remembered something from the night before, something Max and I had discussed in passing as we double-checked the tanks. A manual release valve.\nWithout thinking, I grabbed the walkie-talkie from my belt. 'Max! The valve! Release the pressure! We can boost the balloon higher without needing more hydrogen!'\nThere was a long pause before Max's voice crackled through the speaker. 'What? Are you crazy? That's gonna-'\n'I don't have time for why or how, just do it!' I shouted into the mic. 'Now!'\nI slammed the walkie-talkie down, my heart racing.\nFor a heartbeat, everything stopped. Then came the sound-the unmistakable hiss of gas escaping from the valve. It was like someone had cracked open a dam. But this wasn't a risk-it was our chance.\nThe balloon jerked upward, gaining more lift. I watched in disbelief as it began to climb faster. We had just enough hydrogen to get it airborne, but not enough to make it last as long as we'd hoped. By releasing some pressure, we'd given it a burst-enough to send it higher and faster, without risking a catastrophic failure.\nI turned to the group, eyes wide with adrenaline. 'It's working!' I yelled. 'Everyone-now!'\nMax scrambled to get everyone in position, and in that frantic moment, chaos turned into action. We started securing the final payloads, quickly working as a team. The energy was palpable-everyone had a job, and no one was wasting time.\nThe balloon surged higher, carried by the decision I'd just made on pure instinct. My heart pounded in my ears as I watched it climb into the sky, the bright sun shining off its latex skin. This was it. This was the moment everything hinged on.\nWe hadn't just saved the launch. We had redefined it."
+		(exclude_from_sim no)
+		(at 137.922 -47.498 0)
+		(effects
+			(font
+				(size 1.27 1.27)
+			)
+		)
+	)
 	(text "Interrupt / Wake"
 		(exclude_from_sim no)
@@
 	(wire
 		(pts
-			(xy 265.43 102.87) (xy 245.11 102.87)
+			(xy 266.7 102.87) (xy 245.11 102.87)
 		)
 		(stroke
@@
 	(global_label "CS_BARO TMCU"
 		(shape input)
-		(at 265.43 102.87 0)
+		(at 266.7 102.87 0)
 		(fields_autoplaced yes)
 		(effects
@@
 		)
 		(property "Intersheetrefs" "${INTERSHEET_REFS}"
-			(at 282.8085 102.87 0)
+			(at 284.0785 102.87 0)
 			(effects
 				(font
@@
 	(symbol
 		(lib_id "power:+3.3V")
-		(at 265.43 95.25 0)
+		(at 266.7 95.25 0)
 		(unit 1)
 		(exclude_from_sim no)
@@
 		(dnp no)
 		(property "Reference" "#PWR0112"
-			(at 265.43 99.06 0)
+			(at 266.7 99.06 0)
 			(effects
 				(font
@@
 		)
 		(property "Value" "+3.3V"
-			(at 265.43 89.408 90)
+			(at 266.7 89.408 90)
 			(effects
 				(font
@@
 		)
 		(property "Footprint" ""
-			(at 265.43 95.25 0)
+			(at 266.7 95.25 0)
 			(effects
 				(font
@@
 		)
 		(property "Datasheet" ""
-			(at 265.43 95.25 0)
+			(at 266.7 95.25 0)
 			(effects
 				(font
@@
 		)
 		(property "Description" "Power symbol creates a global label with name \"+3.3V\""
-			(at 265.43 95.25 0)
+			(at 266.7 95.25 0)
 			(effects
 				(font
@@
 	(symbol
 		(lib_id "Device:R")
-		(at 265.43 99.06 0)
+		(at 266.7 99.06 0)
 		(unit 1)
 		(exclude_from_sim no)
@@
 		(dnp no)
 		(property "Reference" "R39"
-			(at 264.668 81.788 0)
+			(at 265.938 81.788 0)
 			(effects
 				(font
@@
 		)
 		(property "Value" "10k"
-			(at 264.668 84.328 0)
+			(at 265.938 84.328 0)
 			(effects
 				(font
@@
 		)
 		(property "Footprint" "Resistor_SMD:R_0603_1608Metric"
-			(at 263.652 99.06 90)
+			(at 264.922 99.06 90)
 			(effects
 				(font
@@
 		)
 		(property "Datasheet" "~"
-			(at 265.43 99.06 0)
+			(at 266.7 99.06 0)
 			(effects
 				(font
@@
 		)
 		(property "Description" "Resistor"
-			(at 265.43 99.06 0)
+			(at 266.7 99.06 0)
 			(effects
 				(font
