File: flight computer/power.kicad_sch (KiCad schematic)
At the start: 29 parts, among them J10 Conn_01x02_Pin, Q2 DMG2301L, U13 LTC4412xS6, U14 TPS61092, U15 AP2112K-3.3, U9 TPS82130

Commit message: wiirng
Parts:
- removed D19: PMEG6020ER, Diode_SMD:Nexperia_CFP3_SOD-123W, symbol Diode:PMEG6020ER
Connections:
- net POWAAAA is gone; now on net VBUS: C28.1, D20.2 (A), Q2.2 (S), U13.6 (SENSE)
Changed lines of the file:
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@@
 	(symbol
 		(lib_id "power:VBUS")
-		(at 148.59 57.15 0)
+		(at 148.59 64.77 0)
 		(unit 1)
 		(exclude_from_sim no)
@@
 		(fields_autoplaced yes)
 		(property "Reference" "#PWR01"
-			(at 148.59 60.96 0)
+			(at 148.59 68.58 0)
 			(effects
 				(font
@@
 		)
 		(property "Value" "VBUS"
-			(at 148.59 52.07 0)
+			(at 148.59 59.69 0)
 			(effects
 				(font
@@
 		)
 		(property "Footprint" ""
-			(at 148.59 57.15 0)
+			(at 148.59 64.77 0)
 			(effects
 				(font
@@
 		)
 		(property "Datasheet" ""
-			(at 148.59 57.15 0)
+			(at 148.59 64.77 0)
 			(effects
 				(font
@@
 		)
 		(property "Description" "Power symbol creates a global label with name \"VBUS\""
-			(at 148.59 57.15 0)
+			(at 148.59 64.77 0)
 			(effects
 				(font
@@
 					(unit 1)
 				)
-			)
-		)
-	)
-	(symbol
-		(lib_id "Diode:PMEG6020ER")
-		(at 148.59 60.96 90)
-		(unit 1)
-		(exclude_from_sim no)
-		(in_bom yes)
-		(on_board yes)
-		(dnp no)
-		(property "Reference" "D19"
-			(at 158.75 58.674 0)
-			(effects
-				(font
-					(size 1.27 1.27)
-				)
-			)
-		)
-		(property "Value" "PMEG6020ER"
-			(at 156.21 58.674 0)
-			(effects
-				(font
-					(size 1.27 1.27)
-				)
-			)
-		)
-		(property "Footprint" "Diode_SMD:Nexperia_CFP3_SOD-123W"
-			(at 153.035 60.96 0)
-			(effects
-				(font
-					(size 1.27 1.27)
-				)
-				(hide yes)
-			)
-		)
-		(property "Datasheet" "https://assets.nexperia.com/documents/data-sheet/PMEG6020ER.pdf"
-			(at 148.59 60.96 0)
-			(effects
-				(font
-					(size 1.27 1.27)
-				)
-				(hide yes)
-			)
-		)
-		(property "Description" "60V, 2A low Vf MEGA Schottky barrier rectifier, SOD-123W"
-			(at 148.59 60.96 0)
-			(effects
-				(font
-					(size 1.27 1.27)
-				)
-				(hide yes)
-			)
-		)
-		(pin "2"
-		)
-		(pin "1"
-		)
-		(instances
-			(project "horizon"
-				(path "/78d9c2f3-deae-418a-8c21-4820ea8fc57f/9f395e7d-f0e3-417c-8bdc-8f8d3cf70e8c"
-					(reference "D19")
-					(unit 1)
-				)

Commit message: periodic commit
Parts:
- removed D23: PMEG6020ER, Diode_SMD:Nexperia_CFP3_SOD-123W, symbol Diode:PMEG6020ER
Connections:
- net +5V: now also C32.1, U9.1 (EN), U9.2 (VIN)
Changed lines of the file:
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@@
+	)
+	(junction
+		(at 154.94 102.87)
+		(diameter 0)
+		(color 0 0 0 0)
 	)
 	(junction
@@
 	(junction
 		(at 240.03 102.87)
-		(diameter 0)
-		(color 0 0 0 0)
-	)
-	(junction
-		(at 154.94 102.87)
 		(diameter 0)
 		(color 0 0 0 0)
@@
 	(wire
 		(pts
+			(xy 154.94 102.87) (xy 163.83 102.87)
+		)
+		(stroke
+			(width 0)
+			(type default)
+		)
+	)
+	(wire
+		(pts
 			(xy 59.69 62.23) (xy 62.23 62.23)
 		)
@@
 		(pts
 			(xy 69.85 62.23) (xy 69.85 59.69)
-		)
-		(stroke
-			(width 0)
-			(type default)
-		)
-	)
-	(wire
-		(pts
-			(xy 162.56 102.87) (xy 163.83 102.87)
 		)
 		(stroke
@@
 					(unit 1)
 				)
-			)
-		)
-	)
-	(symbol
-		(lib_id "Diode:PMEG6020ER")
-		(at 158.75 102.87 180)
-		(unit 1)
-		(exclude_from_sim no)
-		(in_bom yes)
-		(on_board yes)
-		(dnp no)
-		(property "Reference" "D23"
-			(at 154.94 106.172 0)
-			(effects
-				(font
-					(size 1.27 1.27)
-				)
-			)
-		)
-		(property "Value" "PMEG6020ER"
-			(at 154.94 108.712 0)
-			(effects
-				(font
-					(size 1.27 1.27)
-				)
-			)
-		)
-		(property "Footprint" "Diode_SMD:Nexperia_CFP3_SOD-123W"
-			(at 158.75 98.425 0)
-			(effects
-				(font
-					(size 1.27 1.27)
-				)
-				(hide yes)
-			)
-		)
-		(property "Datasheet" "https://assets.nexperia.com/documents/data-sheet/PMEG6020ER.pdf"
-			(at 158.75 102.87 0)
-			(effects
-				(font
-					(size 1.27 1.27)
-				)
-				(hide yes)
-			)
-		)
-		(property "Description" "60V, 2A low Vf MEGA Schottky barrier rectifier, SOD-123W"
-			(at 158.75 102.87 0)
-			(effects
-				(font
-					(size 1.27 1.27)
-				)
-				(hide yes)
-			)
-		)
-		(pin "2"
-		)
-		(pin "1"
-		)
-		(instances
-			(project "horizon"
-				(path "/78d9c2f3-deae-418a-8c21-4820ea8fc57f/9f395e7d-f0e3-417c-8bdc-8f8d3cf70e8c"
-					(reference "D23")
-					(unit 1)
-				)

Commit message: daily commit
Parts:
- J10: footprint Connector_JST:JST_PH_B2B-PH-K_1x02_P2.00mm_Vertical -> TerminalBlock_Phoenix:TerminalBlock_Phoenix_MPT-0,5-2-2.54_1x02_P2.54mm_Horizontal
Changed lines of the file:
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@@
 			)
 		)
-		(property "Footprint" "Connector_JST:JST_PH_B2B-PH-K_1x02_P2.00mm_Vertical"
+		(property "Footprint" "TerminalBlock_Phoenix:TerminalBlock_Phoenix_MPT-0,5-2-2.54_1x02_P2.54mm_Horizontal"
 			(at 26.67 39.37 0)
 			(effects

Commit message: power fixes
Parts:
- removed C29: 10u, Capacitor_SMD:C_0603_1608Metric, symbol Device:C
- removed C30: 2u2, Capacitor_SMD:C_0603_1608Metric, symbol Device:C
- removed C31: 100u, Capacitor_SMD:C_0603_1608Metric, symbol Device:C_Polarized_US
- removed L2: SLF7055T-6R8N2R8-3PF, Inductor_SMD:L_7.3x7.3_H4.5, symbol SLF7055T-6R8N2R8-3PF[1]:SLF7055T-6R8N2R8-3PF
- removed R40, R41: 100k, Resistor_SMD:R_0603_1608Metric, symbol Device:R
- removed U14: TPS61092, Package_DFN_QFN:Texas_RSA_VQFN-16-1EP_4x4mm_P0.65mm_EP2.7x2.7mm_ThermalVias, symbol Regulator_Switching:TPS61092
- added C21, C24, C25: 10uF, Capacitor_SMD:C_0603_1608Metric, symbol Device:C
- added C22: 1uF, Capacitor_SMD:C_0603_1608Metric, symbol Device:C
- added L2: 2.2uH, Inductor_SMD:L_APV_ANR4018, symbol Device:L
- added U3: TPS61200DRC, Package_SON:Texas_S-PVSON-N10_ThermalVias, symbol Regulator_Switching:TPS61200DRC
- R42: value 430k -> 900k
Connections:
- net GND: now also C21.2, C22.2, C24.2, C25.2, U3.11 (PAD), U3.4 (PGND), U3.9 (GND)
- net bat: now also C24.1, C25.1, U3.2 (VOUT)
- net at J10.1 (Pin_1): now also C21.1, L2.1, U3.5 (VIN), U3.6 (EN), U3.7 (UVLO), U3.8 (PS)
- net at R42.2, R43.1: now also U3.10 (FB)
- new net: C22.1, U3.1 (VAUX)
- new net: L2.2, U3.3 (L)
- no-connect marks 3 -> 2
Other:
- moved on the sheet: J10, R42, R43

Commit message: if this breaks stuff womp womp
Other:
- note added: "3.6v"
- note added: "5v"
Changed lines of the file:
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@@
 	(generator_version "9.0")
 	(paper "A4")
+	(text "5v"
+		(exclude_from_sim no)
+		(at 169.672 66.04 0)
+		(effects
+			(font
+				(size 1.27 1.27)
+			)
+		)
+	)
+	(text "5v"
+		(exclude_from_sim no)
+		(at 137.414 100.584 0)
+		(effects
+			(font
+				(size 1.27 1.27)
+			)
+		)
+	)
+	(text "3.6v"
+		(exclude_from_sim no)
+		(at 223.52 101.6 0)
+		(effects
+			(font
+				(size 1.27 1.27)
+			)
+		)
+	)
 	(junction
 		(at 213.36 102.87)

Commit message: bluetooth, gps, gyro reviewed - doing pressure tmrw
Changed lines of the file:
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@@
+		)
+	)
+	(text "5v"
+		(exclude_from_sim no)
+		(at 117.602 35.306 0)
+		(effects
+			(font
+				(size 1.27 1.27)
+			)
 		)
 	)
